File: proto1.sch (KiCad schematic (older format))
At the start: 12 parts, among them P1 sw, P2 BR-LED, P3 Solar panel, P4 BAT, Q1 7000

Commit message: motion sensing hack added
Parts:
- added D?: LED, Headers:Pin_Header_Straight_1x02, symbol LED
- added FET: 2N7000, TO92:TO-92_Inline_Narrow_Oval, symbol Q_NMOS_SGD
- added P?: - 4V BATTERY +, MyLib:bat-LA, symbol CONN_01X02
- added R?: 47, Discret:R3, symbol R
- P2: value BR-LED -> BRIGHT-LED
- P4: value BAT -> - 4V BATTERY +
Connections:
- new net: D?.1 (K), FET.3 (D)
- new net: D?.2 (A), R?.2
- new net +: P?.2 (P2), R?.1
- new net -: FET.1 (S), P?.1 (P1)
- new net OUTPUT: FET.2 (G)
Other:
- note added: "MOTION DETECTOR HACK"
- note added: "MOTION SENSOR (SR-501)"
- note added: "SOLAR GARDEN LAMP\n"
Changed lines of the file:
@@
 P 1650 3975
 F 0 "P4" H 1650 4125 50  0000 C CNN
-F 1 "BAT" V 1750 3975 50  0000 C CNN
+F 1 "- 4V BATTERY +" V 1750 3975 50  0000 C CNN
 F 2 "MyLib:bat-LA" H 1650 3975 60  0001 C CNN
 F 3 "" H 1650 3975 60  0000 C CNN
@@
 P 1050 3950
 F 0 "P2" H 1050 4100 50  0000 C CNN
-F 1 "BR-LED" V 1150 3950 50  0000 C CNN
+F 1 "BRIGHT-LED" V 1150 3950 50  0000 C CNN
 F 2 "Headers:Pin_Header_Straight_1x02" H 1050 3950 60  0001 C CNN
 F 3 "" H 1050 3950 60  0000 C CNN
@@
 Wire Wire Line
 	2425 3350 2425 3225
+Text Notes 1930 2795 0    60   ~ 0
+SOLAR GARDEN LAMP\n
+Text Notes 1820 5185 0    60   ~ 0
+MOTION DETECTOR HACK
+$Comp
+L CONN_01X02 P?
+U 1 1 58183299
+P 1585 5740
+F 0 "P?" H 1585 5890 50  0000 C CNN
+F 1 "- 4V BATTERY +" V 1685 5740 50  0000 C CNN
+F 2 "MyLib:bat-LA" H 1585 5740 60  0001 C CNN
+F 3 "" H 1585 5740 60  0000 C CNN
+	1    1585 5740
+	-1   0    0    1
+$EndComp
+$Comp
+L Q_NMOS_SGD FET
+U 1 1 58183338
+P 3200 5785
+F 0 "FET" H 3565 5810 50  0000 R CNN
+F 1 "2N7000" H 3640 5720 50  0000 R CNN
+F 2 "TO92:TO-92_Inline_Narrow_Oval" H 3400 5885 29  0001 C CNN
+F 3 "" H 3200 5785 60  0000 C CNN
+	1    3200 5785
+	1    0    0    -1
+$EndComp
+$Comp
+L LED D?
+U 1 1 5818346E
+P 3030 5445
+F 0 "D?" H 2980 5345 50  0000 C CNN
+F 1 "LED" H 3045 5340 50  0000 C CNN
+F 2 "Headers:Pin_Header_Straight_1x02" H 3030 5445 60  0001 C CNN
+F 3 "" H 3030 5445 60  0000 C CNN
+	1    3030 5445
+	-1   0    0    1
+$EndComp
+$Comp
+L R R?
+U 1 1 58183922
+P 2550 5445
+F 0 "R?" V 2630 5445 50  0000 C CNN
+F 1 "47" V 2550 5445 50  0000 C CNN
+F 2 "Discret:R3" V 2480 5445 30  0001 C CNN
+F 3 "" H 2550 5445 30  0000 C CNN
+	1    2550 5445
+	0    -1   -1   0
+$EndComp
+Wire Wire Line
+	2700 5445 2830 5445
+Wire Wire Line
+	3230 5445 3300 5445
+Wire Wire Line
+	3300 5445 3300 5585
+Wire Wire Line
+	1785 5690 1785 5445
+Wire Wire Line
+	1785 5445 2400 5445
+Wire Wire Line
+	1785 5790 1785 5985
+Wire Wire Line
+	1785 5985 3300 5985
+Text GLabel 2240 5640 0    60   Input ~ 0
++
+Text GLabel 2245 5885 0    60   Input ~ 0
+-
+Text GLabel 2505 5760 0    60   Input ~ 0
+OUTPUT
+Wire Wire Line
+	2240 5640 2240 5445
+Connection ~ 2240 5445
+Wire Wire Line
+	2245 5885 2245 5985
+Connection ~ 2245 5985
+Wire Wire Line
+	2505 5760 3000 5760
+Wire Wire Line
+	3000 5760 3000 5785
+Wire Bus Line
+	2035 5570 2035 6095
+Wire Bus Line
+	2035 6095 2620 6095
+Wire Bus Line
+	2620 6095 2620 5530
+Wire Bus Line
+	2620 5530 2015 5530
+Wire Bus Line
+	2015 5530 2015 5570
+Wire Bus Line
+	2015 5570 2035 5570
+Text Notes 1785 6240 0    60   ~ 0
+MOTION SENSOR (SR-501)
 $EndSCHEMATC
